File: PCB Design/ECG/ECG.kicad_sch (KiCad schematic)
At the start: 39 parts

Commit message: schem done, pcb 50%
Parts:
- removed C?: 10uF, symbol Device:C
- removed SW?: SW_Push, Buttons:Tactile_pushbutton_6x6mm, symbol Switch:SW_Push
- removed U?: Li-Po, Battery_solder_pads:Battery Solder Pad 2.5x2.0mm, symbol Battery:Li-Po
- removed U?: RT5760A, Package_TO_SOT_SMD:SOT-563, symbol RT5760A:RT5760A
- removed U?: 3V3TP, symbol Test points:TP
- removed U?: 5V Switch, Switches:5V, symbol battery switch:Battery_Switch
- removed U?: TP4056M, Package_SO:MSOP-8-1EP_3x3mm_P0.65mm_EP2.5x3mm_Mask1.73x2.36mm_ThermalVias, symbol TP4056M-C21417:TP4056M
- added C12, C13: 100nF, Capacitor_SMD:C_0603_1608Metric_Pad1.08x0.95mm_HandSolder, symbol Device:C
- added J2: JST_01x04_Male, Connector_PinHeader_2.54mm:PinHeader_1x04_P2.54mm_Horizontal, symbol Connector:Conn_01x04_Male
- added TP1, TP2, TP3, TP4: TestPoint_Flag, symbol Connector:TestPoint_Flag
- added TP5: TP Output, TestPoint:TestPoint_Loop_D1.80mm_Drill1.0mm_Beaded, symbol Connector:TestPoint
- added TP6: TP 3V3, TestPoint:TestPoint_Loop_D1.80mm_Drill1.0mm_Beaded, symbol Connector:TestPoint
- added TP7: TP GND, TestPoint:TestPoint_Loop_D1.80mm_Drill1.0mm_Beaded, symbol Connector:TestPoint
- added TP8: TP 5V, TestPoint:TestPoint_Loop_D1.80mm_Drill1.0mm_Beaded, symbol Connector:TestPoint
- added TP9: TP 4V, TestPoint:TestPoint_Loop_D1.80mm_Drill1.0mm_Beaded, symbol Connector:TestPoint
- added U1: Li-Po, Battery_solder_pads:Battery Solder Pad 2.5x2.0mm, symbol Battery:Li-Po
- added U2: TP4056-C21417, Package_SO:MSOP-8-1EP_3x3mm_P0.65mm_EP2.5x3mm_Mask1.73x2.36mm_ThermalVias, symbol TP4056M-C21417:TP4056-C21417
- added U5: 5V_switch, Switches:5V, symbol battery switch:5V_switch
- added U6: TLV62568DBV, Package_TO_SOT_SMD:SOT-23-5, symbol Regulator_Switching:TLV62568DBV
- added U8: Tactile_push_button_6x6mm, Buttons:Tactile_pushbutton_6x6mm, symbol Tactile button:Tactile_push_button_6x6mm
- C1, C11, C2, C3, C5, C8, C9: renamed from C?; footprint (none) -> Capacitor_SMD:C_0603_1608Metric_Pad1.08x0.95mm_HandSolder
- C10: renamed from C?; value 0.1uF -> 100nF; footprint (none) -> Capacitor_SMD:C_0603_1608Metric_Pad1.08x0.95mm_HandSolder
- C6: renamed from C?; value 0.1uF -> 4.7uF; footprint (none) -> Capacitor_SMD:C_0603_1608Metric_Pad1.08x0.95mm_HandSolder
- C7: renamed from C?; value Cff -> 10pF; footprint (none) -> Capacitor_SMD:C_0805_2012Metric_Pad1.18x1.45mm_HandSolder
- D1, D2, D4: renamed from D?; footprint (none) -> LED_SMD:LED_0603_1608Metric
- J1: renamed from J?; value Conn_01x05_Female -> 01x05_Female
- L1: renamed from L?; value 1uH -> 2.2uH; footprint (none) -> Inductor:CY43-2.2uH
- R1, R10, R2, R3, R4, R5, R6, R7, R8, R9: renamed from R?; footprint (none) -> Resistor_SMD:R_0805_2012Metric_Pad1.20x1.40mm_HandSolder
- Rprog1: renamed from Rprog; footprint (none) -> Resistor_SMD:R_0805_2012Metric_Pad1.20x1.40mm_HandSolder
- U10: renamed from U?; footprint XCVR_ESP32-C3-MINI-1-N4 -> ESP32:XCVR_ESP32-C3-MINI-1-N4
- U9: renamed from U?; footprint (none) -> USBS:HRO_TYPE-C-31-M-12
- gave numbers to parts that had none: 4
Connections:
- net +3V3: now also J2.1 (Pin_1), TP2.1, TP6.1, U8.4
- net +4V: now also C13.1, TP9.1, U6.1 (EN), U6.4 (VIN)
- net +5V: now also C12.1, U2.8 (CE), U5.1; no longer C11.1, U9.A4_B9 (VBUS), U9.B4_A9 (VBUS)
- net +BATT: now also C13.2, U2.5 (BAT)
- net BTN: now also U8.1
- net BatO: now also U1.1 (+Bat)
- net In_5V: now also C11.1, U9.A4_B9 (VBUS), U9.B4_A9 (VBUS), C12.2, TP4.1, TP8.1, U2.4 (VCC), U5.2
- net Output: now also TP1.1, TP5.1
- net at Rprog1.1: now also U2.2 (PROG)
- net at D1.1 (K): now also U2.7 (CHRG)
- net at C7.2, R5.2, R6.1: now also U6.5 (FB)
- net at L1.1: now also U6.3 (SW)
- net at D2.1 (K): now also U2.6 (STDBY)
- net RX: now reaches U10.30 (RXD0)
- net RX: now also J2.3 (Pin_3)
- net TX: now reaches U10.31 (TXD0)
- net TX: now also J2.2 (Pin_2)
- net -BATT renamed GND
- net GND: now also J2.4 (Pin_4), TP3.1, TP7.1, U1.2 (-Bat), U2.1 (TEMP), U2.3 (GND), U6.2 (GND)
- no-connect marks 28 -> 29
Other:
- note added: "RX TX"
- moved on the sheet: C1, C2, C5, C6, C7, C8, D4, J1, L1, R1, R4, R5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
